Commit message: Update frames.
Signed-off-by: Benjamin Perseghetti <bperseghetti@rudislabs.com>

File: elm4_description/urdf/elm4.urdf (robot description, URDF)
Before this commit: robot elm4, 4 links, 3 joints
Joints:
- joint base_joint: origin xyz=0.0 0.0 0.0 rpy=0 0 0 -> xyz=0.0 0.0 -.15 rpy=0 0 0
- joint rplidar_joint: origin xyz=0 0 .715 rpy=0 0 0 -> xyz=0 0 .22 rpy=0 0 0

Commit message: Update to use general lidar.
Signed-off-by: Benjamin Perseghetti <bperseghetti@rudislabs.com>

File: elm4_description/urdf/elm4.urdf (robot description, URDF)
Before this commit: robot elm4, 4 links, 3 joints
Links:
- removed link /link/rplidar_link/sensor/rplidar/scan
- removed link rplidar_link
- added link /link/lidar_link/sensor/lidar/scan
- added link lidar_link; visual mesh filename=package://elm4_description/meshes/rplidar.dae scale=1 1 1
Joints:
- removed joint rplidar_joint
- removed joint rplidar_joint2
- added joint lidar_joint0: type fixed, parent base_link, child lidar_link, origin xyz=0 0 .22 rpy=0 0 0
- added joint lidar_joint2: type fixed, parent lidar_link, child /link/lidar_link/sensor/lidar/scan, origin xyz=0.0 0.0 0.0 rpy=0 0 0

Commit message: Update lidar to stl27l.
Signed-off-by: Benjamin Perseghetti <bperseghetti@rudislabs.com>

File: elm4_description/urdf/elm4.urdf (robot description, URDF)
Before this commit: robot elm4, 4 links, 3 joints
Links:
- link lidar_link: geometry visual mesh filename=package://elm4_description/meshes/STL27L.dae scale=1 1 1
Joints:
- joint lidar_joint0: origin xyz=0 0 .22 rpy=0 0 0 -> xyz=0 0 .2 rpy=0 0 0
